Commit message: Camera added

File: turtlebot3_description/urdf/turtlebot3_burger.urdf.xacro (robot description, xacro)
@@ -140,3 +140,44 @@
     </inertial>
   </link>
+  <!-- Camera -->
+  <joint type="fixed" name="camera_joint">
+    <origin xyz="0.03 0 0.11" rpy="0 0.79 0"/>
+    <child link="camera_link"/>
+    <parent link="base_link"/>
+    <axis xyz="0 1 0" />
+  </joint>
+  <link name='camera_link'>
+    <pose>0 0 0 0 0 0</pose>
+    <inertial>
+      <mass value="0.001"/>
+      <origin xyz="0 0 0" rpy="0 0 0"/>
+      <inertia
+          ixx="1e-6" ixy="0" ixz="0"
+          iyy="1e-6" iyz="0"
+          izz="1e-6"
+      />
+    </inertial>
+    <collision name='collision'>
+      <origin xyz="0 0 0" rpy="0 0 0"/>
+      <geometry>
+        <box size=".01 .01 .01"/>
+      </geometry>
+    </collision>
+    <visual name='camera_link_visual'>
+      <origin xyz="0 0 0" rpy="0 0 0"/>
+      <geometry>
+        <box size=".02 .02 .02"/>
+      </geometry>
+    </visual>
+  </link>
+  <gazebo reference="camera_link">
+    <material>Gazebo/Red</material>
+  </gazebo>
+  <joint type="fixed" name="camera_optical_joint">
+    <origin xyz="0 0 0" rpy="-1.5707 0 -1.5707"/>
+    <child link="camera_link_optical"/>
+    <parent link="camera_link"/>
+  </joint>
+  <link name="camera_link_optical">
+  </link>
 </robot>

Commit message: Kamera megfelelo pozicio megadas

File: turtlebot3_description/urdf/turtlebot3_burger.urdf.xacro (robot description, xacro)
@@ -142,5 +142,5 @@
   <!-- Camera -->
   <joint type="fixed" name="camera_joint">
-    <origin xyz="0.03 0 0.11" rpy="0 0.79 0"/>
+    <origin xyz="0.03 0 0.11" rpy="0 -0.15 0"/>
     <child link="camera_link"/>
     <parent link="base_link"/>
